Commit message: Add gazebo control to urdf macro

File: lab09_gazebo/urdf/inc/ur5e_macro.xacro (robot description, xacro)
@@ -5,28 +5,60 @@
     for the various "parameters files" parameters for a UR5e.
     File copied from the fmauch_universal_robot repository and modified
-  -->
-  <xacro:macro name="ur5e_robot" params="
-      prefix
-      joint_limits_parameters_file:='$(find lab09_gazebo)/config/ur5e/joint_limits.yaml'
-      kinematics_parameters_file:='$(find ur_description)/config/ur5e/default_kinematics.yaml'
-      physical_parameters_file:='$(find ur_description)/config/ur5e/physical_parameters.yaml'
-      visual_parameters_file:='$(find ur_description)/config/ur5e/visual_parameters.yaml'
-      transmission_hw_interface:=hardware_interface/PositionJointInterface
-      safety_limits:=false
-      safety_pos_margin:=0.15
-      safety_k_position:=20"
-      >
-      <xacro:include filename="$(find ur_description)/urdf/inc/ur_macro.xacro"/>
-      <xacro:ur_robot
-          prefix="${prefix}"
-          joint_limits_parameters_file="${joint_limits_parameters_file}"
-          kinematics_parameters_file="${kinematics_parameters_file}"
-          physical_parameters_file="${physical_parameters_file}"
-          visual_parameters_file="${visual_parameters_file}"
-          transmission_hw_interface="${transmission_hw_interface}"
-          safety_limits="${safety_limits}"
-          safety_pos_margin="${safety_pos_margin}"
-          safety_k_position="${safety_k_position}"
-          />
-  </xacro:macro>
+    -->
+    <xacro:macro name="ur5e_robot" params="
+        prefix
+        joint_limits_parameters_file:='$(find lab09_gazebo)/config/ur5e/joint_limits.yaml'
+        kinematics_parameters_file:='$(find ur_description)/config/ur5e/default_kinematics.yaml'
+        physical_parameters_file:='$(find ur_description)/config/ur5e/physical_parameters.yaml'
+        visual_parameters_file:='$(find ur_description)/config/ur5e/visual_parameters.yaml'
+        transmission_hw_interface:=hardware_interface/PositionJointInterface
+        safety_limits:=false
+        safety_pos_margin:=0.15
+        safety_k_position:=20"
+        >
+        <xacro:include filename="$(find ur_description)/urdf/inc/ur_macro.xacro"/>
+        <xacro:ur_robot
+            prefix="${prefix}"
+            joint_limits_parameters_file="${joint_limits_parameters_file}"
+            kinematics_parameters_file="${kinematics_parameters_file}"
+            physical_parameters_file="${physical_parameters_file}"
+            visual_parameters_file="${visual_parameters_file}"
+            transmission_hw_interface="${transmission_hw_interface}"
+            safety_limits="${safety_limits}"
+            safety_pos_margin="${safety_pos_margin}"
+            safety_k_position="${safety_k_position}"
+            />
+        <!-- Configure self collision properties per link -->
+        <gazebo reference="${prefix}shoulder_link">
+            <selfCollide>true</selfCollide>
+        </gazebo>
+        <gazebo reference="${prefix}upper_arm_link">
+            <selfCollide>true</selfCollide>
+        </gazebo>
+        <gazebo reference="${prefix}forearm_link">
+            <selfCollide>true</selfCollide>
+        </gazebo>
+        <gazebo reference="${prefix}wrist_1_link">
+            <selfCollide>true</selfCollide>
+        </gazebo>
+        <gazebo reference="${prefix}wrist_3_link">
+            <selfCollide>true</selfCollide>
+        </gazebo>
+        <gazebo reference="${prefix}wrist_2_link">
+            <selfCollide>true</selfCollide>
+        </gazebo>
+        <gazebo reference="${prefix}ee_link">
+            <selfCollide>true</selfCollide>
+        </gazebo>
+        <!--
+          Inject Gazebo ROS Control plugin, which allows us to use ros_control
+          controllers to control the virtual robot hw.
+        -->
+        <gazebo>
+            <plugin name="ros_control" filename="libgazebo_ros_control.so">
+                <!--robotNamespace>/</robotNamespace-->
+            <!--robotSimType>gazebo_ros_control/DefaultRobotHWSim</robotSimType-->
+    </plugin>
+</gazebo>
+    </xacro:macro>
 </robot>
