Commit message: Add missing files

File: lab09_gazebo/urdf/inc/robotiq_epick_model.xacro (robot description, xacro)
@@ -45,5 +45,5 @@
     </collision>  -->
   </link>
-  <joint name="epick_end_effector_joint" type="revolute">
+  <joint name="epick_end_effector_joint" type="fixed">
       <axis xyz="1 0 0" />
     <parent link="epick"/>
