Commit message: Move correctly but doesn't pick up box

File: lab09_gazebo/urdf/inc/robotiq_epick.gazebo.xacro (robot description, xacro)
@@ -8,6 +8,6 @@
         <bodyName>epick_end_effector</bodyName>
         <topicName>grasping</topicName>
-        <maxForce>150</maxForce>
-        <maxDistance>0.03</maxDistance>
+        <maxForce>250</maxForce>
+        <maxDistance>0.05</maxDistance>
         <minDistance>0.01</minDistance>
       </plugin>

File: lab09_gazebo/urdf/inc/robotiq_epick_model.xacro (robot description, xacro)
@@ -45,5 +45,5 @@
     </collision>  -->
   </link>
-  <joint name="epick_end_effector_joint" type="fixed">
+  <joint name="epick_end_effector_joint" type="revolute">
       <axis xyz="1 0 0" />
     <parent link="epick"/>

File: ur5e_epick_moveit_config/urdf/ur5e_epick_auto_gen.urdf (robot description, URDF)
Before this commit: robot ur5e_epick, 13 links, 12 joints
Joints:
- joint epick_end_effector_joint: type fixed -> revolute
