Commit message: epick in gazebo

File: lab09_gazebo/urdf/ur5e_robotiq_epick_robot.urdf.xacro (robot description, xacro)
@@ -6,6 +6,6 @@
   <!-- ur5e -->
   <!-- TODO: have this variable based on limited == true/false -->
-  <xacro:include filename="$(find lab09_gazebo)/urdf/inc/ur5e_macro.xacro" />
-  <xacro:ur5e_robot prefix="" />
+  <!-- <xacro:include filename="$(find lab09_gazebo)/urdf/inc/ur5e_macro.xacro" /> -->
+  <!-- <xacro:ur5e_robot prefix="" /> -->
   <!-- gripper -->
   <xacro:include filename="$(find lab09_gazebo)/urdf/inc/robotiq_epick_model.xacro" />
@@ -13,16 +13,16 @@
   <joint name="world_joint" type="fixed">
     <parent link="world" />
-    <child link = "base_link" />
-    <origin xyz="0.8 0.0 0.675" rpy="0.0 0.0 0.0" />
+    <child link = "epick" />
+    <origin xyz="0.0 0.0 0.0" rpy="0.0 0.0 0.0" />
   </joint>
-  <joint name="robotiq_epick_joint" type="fixed">
-    <origin xyz="0 0 0.004" rpy="0 0 ${-pi/2.0}" />
-    <parent link="tool0"/>
-    <child link="epick"/>
-  </joint>
-  <joint name="camera_joint" type="fixed">
-    <parent link="world" />
-    <child link = "camera_link" />
-    <origin xyz="1.9 0.25 1.675" rpy="0.0 ${pi/2.6} ${pi}" />
-  </joint>
+  <!-- <joint name="world_joint" type="fixed"> -->
+  <!--   <parent link="world" /> -->
+  <!--   <child link = "base_link" /> -->
+  <!--   <origin xyz="0.8 0.0 0.675" rpy="0.0 0.0 0.0" /> -->
+  <!-- </joint> -->
+  <!-- <joint name="robotiq_epick_joint" type="fixed"> -->
+  <!--   <origin xyz="0 0 0.004" rpy="0 0 ${-pi/2.0}" /> -->
+  <!--   <parent link="tool0"/> -->
+  <!--   <child link="epick"/> -->
+  <!-- </joint> -->
 </robot>

Commit message: ur5e with epick in world

File: lab09_gazebo/urdf/ur5e_robotiq_epick_robot.urdf.xacro (robot description, xacro)
@@ -2,27 +2,13 @@
 <robot xmlns:xacro="http://ros.org/wiki/xacro"
        name="ur5e" >
-  <!-- <!-1- common stuff -1-> -->
-  <!-- <xacro:include filename="$(find ur_description)/urdf/common.gazebo.xacro" /> -->
-  <!-- ur5e -->
-  <!-- TODO: have this variable based on limited == true/false -->
-  <!-- <xacro:include filename="$(find lab09_gazebo)/urdf/inc/ur5e_macro.xacro" /> -->
-  <!-- <xacro:ur5e_robot prefix="" /> -->
-  <!-- gripper -->
-  <xacro:include filename="$(find lab09_gazebo)/urdf/inc/robotiq_epick_model.xacro" />
+  <!-- ur5e with epick -->
+  <xacro:include filename="$(find lab09_gazebo)/urdf/inc/ur5e_epick.urdf.xacro" />
+  <!-- Root link -->
   <link name="world" />
+  <!-- fix robot to world -->
   <joint name="world_joint" type="fixed">
     <parent link="world" />
-    <child link = "epick" />
-    <origin xyz="0.0 0.0 0.0" rpy="0.0 0.0 0.0" />
+    <child link = "base_link" />
+    <origin xyz="0.8 0.0 0.775" rpy="0.0 0.0 0.0" />
   </joint>
-  <!-- <joint name="world_joint" type="fixed"> -->
-  <!--   <parent link="world" /> -->
-  <!--   <child link = "base_link" /> -->
-  <!--   <origin xyz="0.8 0.0 0.675" rpy="0.0 0.0 0.0" /> -->
-  <!-- </joint> -->
-  <!-- <joint name="robotiq_epick_joint" type="fixed"> -->
-  <!--   <origin xyz="0 0 0.004" rpy="0 0 ${-pi/2.0}" /> -->
-  <!--   <parent link="tool0"/> -->
-  <!--   <child link="epick"/> -->
-  <!-- </joint> -->
 </robot>

Commit message: Robot in gazebo 'fixed' to table and controlled by moveit

File: lab09_gazebo/urdf/ur5e_robotiq_epick_robot.urdf.xacro (robot description, xacro)
@@ -1,14 +1,22 @@
 <?xml version="1.0"?>
 <robot xmlns:xacro="http://ros.org/wiki/xacro"
-       name="ur5e_epick" >
-  <!-- ur5e with epick -->
-  <xacro:include filename="$(find lab09_gazebo)/urdf/inc/ur5e_epick.urdf.xacro" />
-  <!-- Root link -->
-  <link name="world" />
-  <!-- fix robot to world -->
-  <joint name="world_joint" type="fixed">
-    <parent link="world" />
-    <child link = "base_link" />
-    <origin xyz="0.8 0.0 0.775" rpy="0.0 0.0 0.0" />
-  </joint>
+    name="ur5e_epick" >
+    <!-- ur5e -->
+    <xacro:include filename="$(find lab09_gazebo)/urdf/inc/ur5e_macro.xacro" />
+    <xacro:ur5e_robot prefix="" />
+    <!-- gripper -->
+    <xacro:include filename="$(find lab09_gazebo)/urdf/inc/robotiq_epick_model.xacro" />
+    <!-- Root link -->
+    <link name="world" />
+    <!-- fix robot to world -->
+    <joint name="world_joint" type="fixed">
+        <parent link="world" />
+        <child link="base_link" />
+    </joint>
+    <!-- fix epick to robot -->
+    <joint name="robotiq_epick_joint" type="fixed">
+        <origin xyz="0 0 0.004" rpy="0 0 ${-pi/2.0}" />
+        <parent link="tool0"/>
+        <child link="epick"/>
+    </joint>
 </robot>
